Commit message: kinetic testing

File: urdf/catvehicle_2_lidars.xacro (robot description, xacro)
@@ -363,5 +363,5 @@
     </inertial>
 </link>
-<!--joint name="camera_joint" type="fixed">
+<joint name="camera_joint" type="fixed">
 <origin xyz="0 0 ${0.725 + sensor_box/2 + 1.25}" rpy="0 0 0"/>
 	<axis xyz="0 0 1"/>
@@ -388,5 +388,5 @@
       <inertia ixx="1e-6" ixy="0" ixz="0" iyy="1e-6" iyz="0" izz="1e-6" />
     </inertial>
-</link-->
+</link>
 <!--Velodyne LIDAR-->
 <!--joint name="velodyne_joint" type="fixed">
